File: Hardware/cell.brd (EAGLE design)
At the start: 44.1 x 44.6 mm, 17 parts, among them T1 Si1013, X1 22-23-2021

Commit message: Formatting
Parts:
- removed X1: 22-23-2021, con-molex:22-23-2021
- added C2: 0.33uF, rcl:C0603
- added IC1: NCV78M05BDTRKG, linear:DPACK_3
- moved C1 5.34 mm to (21.6, 90.9)
- moved R7 5.34 mm to (26.2, 91.5)
- moved D1 5.34 mm to (22.8, 93.1)
Connections:
- removed net VIN: U$1.VIN, X1.1
- new net 5V: IC1.3, U$1.VIN
- new net N$6: C2.1, IC1.1
- net GND: now also C2.2, IC1.4; no longer X1.2
Routing:
- net RX1: track 0.00 -> 26.7 mm
- net TX1: track 0.00 -> 21.7 mm
- net V_BCKP: track 32.0 -> 30.0 mm
- net +3V3: track 67.2 -> 69.1 mm
Other:
- board size 44.1 x 44.6 mm -> 44.1 x 45.9 mm
