File: Hardware/cell.sch (EAGLE design)
At the start: 17 parts, among them T1 Si1013, X1 22-23-2021

Commit message: Formatting
Parts:
- removed X1: 22-23-2021, con-molex:22-23-2021
- added C2: 0.33uF, rcl:C-USC0603
- added IC1: NCV78M05BDTRKG, linear:NCV78M05BDTRKG
Connections:
- removed net VIN: U$1.VIN, X1-1.S
- new net 5V: IC1.VO, U$1.VIN
- new net N$6: C2.1, IC1.VI
- net GND: now also C2.2, IC1.GND; no longer X1-2.S
Changed lines of the file:
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@@
 <?xml version="1.0" encoding="utf-8"?>
 <!DOCTYPE eagle SYSTEM "eagle.dtd">
-<eagle version="9.2.2">
+<eagle version="9.3.0">
 <drawing>
 <settings>
-<setting alwaysvectorfont="yes"/>
+<setting alwaysvectorfont="no"/>
 <setting verticaltext="up"/>
 </settings>
@@
 <part name="GND5" library="supply1" library_urn="urn:adsk.eagle:library:371" deviceset="GND" device=""/>
 <part name="COIN" library="adafruit" deviceset="CR1220" device="SMT" value="CR1220SMD"/>
-<part name="X1" library="con-molex" library_urn="urn:adsk.eagle:library:165" deviceset="22-23-2021" device=""/>
+<part name="GND6" library="supply1" library_urn="urn:adsk.eagle:library:371" deviceset="GND" device=""/>
+<part name="IC1" library="linear" library_urn="urn:adsk.eagle:library:262" deviceset="NCV78M" device="" package3d_urn="urn:adsk.eagle:package:16495/2" technology="05BDTRKG"/>
+<part name="C2" library="rcl" library_urn="urn:adsk.eagle:library:334" deviceset="C-US" device="C0603" package3d_urn="urn:adsk.eagle:package:23616/2" value="0.33uF"/>
 </parts>
 <sheets>
@@
 <attribute name="VALUE" x="119.38" y="181.61" size="1.778" layer="96" rot="R90"/>
 </instance>
-<instance part="X1" gate="-1" x="144.78" y="180.34" smashed="yes">
-<attribute name="NAME" x="147.32" y="179.578" size="1.524" layer="95"/>
-<attribute name="VALUE" x="144.018" y="181.737" size="1.778" layer="96"/>
-</instance>
-<instance part="X1" gate="-2" x="144.78" y="177.8" smashed="yes">
-<attribute name="NAME" x="147.32" y="177.038" size="1.524" layer="95"/>
+<instance part="GND6" gate="1" x="144.78" y="165.1" smashed="yes">
+<attribute name="VALUE" x="142.24" y="162.56" size="1.778" layer="96"/>
+</instance>
+<instance part="IC1" gate="G$1" x="157.48" y="182.88" smashed="yes">
+<attribute name="NAME" x="149.86" y="188.595" size="1.778" layer="95"/>
+<attribute name="VALUE" x="149.86" y="186.055" size="1.778" layer="96"/>
+</instance>
+<instance part="C2" gate="G$1" x="144.78" y="177.8" smashed="yes">
+<attribute name="NAME" x="145.796" y="178.435" size="1.778" layer="95"/>
+<attribute name="VALUE" x="145.796" y="173.609" size="1.778" layer="96"/>
 </instance>
 </instances>
@@
 </segment>
 <segment>
-<pinref part="X1" gate="-2" pin="S"/>
-<wire x1="142.24" y1="177.8" x2="139.7" y2="177.8" width="0.1524" layer="91"/>
-<label x="139.7" y="177.8" size="1.27" layer="95" rot="R180" xref="yes"/>
+<pinref part="GND6" gate="1" pin="GND"/>
+<pinref part="IC1" gate="G$1" pin="GND"/>
+<wire x1="144.78" y1="170.18" x2="144.78" y2="167.64" width="0.1524" layer="91"/>
+<wire x1="144.78" y1="170.18" x2="157.48" y2="170.18" width="0.1524" layer="91"/>
+<wire x1="157.48" y1="170.18" x2="157.48" y2="175.26" width="0.1524" layer="91"/>
+<wire x1="139.7" y1="170.18" x2="144.78" y2="170.18" width="0.1524" layer="91"/>
+<junction x="144.78" y="170.18"/>
+<pinref part="C2" gate="G$1" pin="2"/>
+<wire x1="144.78" y1="172.72" x2="144.78" y2="170.18" width="0.1524" layer="91"/>
 </segment>
 </net>
@@
 </segment>
 </net>
-<net name="VIN" class="0">
+<net name="N$9" class="0">
+<segment>
+<junction x="71.12" y="83.82"/>
+</segment>
+</net>
+<net name="N$10" class="0">
+<segment>
+<pinref part="LED1" gate="G$1" pin="A"/>
+<pinref part="R1" gate="G$1" pin="1"/>
+<wire x1="25.4" y1="157.48" x2="27.94" y2="157.48" width="0.1524" layer="91"/>
+</segment>
+</net>
+<net name="N$2" class="0">
+<segment>
+<pinref part="R1" gate="G$1" pin="2"/>
+<pinref part="U$1" gate="G$1" pin="14/A0"/>
+<wire x1="38.1" y1="157.48" x2="48.26" y2="157.48" width="0.1524" layer="91" style="longdash"/>
+</segment>
+</net>
+<net name="N$13" class="0">
+<segment>
+<pinref part="R7" gate="G$1" pin="2"/>
+<pinref part="C1" gate="G$1" pin="3V3"/>
+<wire x1="-30.48" y1="50.8" x2="-30.48" y2="45.72" width="0.1524" layer="91" style="longdash"/>
+</segment>
+</net>
+<net name="N$12" class="0">
+<segment>
+<pinref part="U$1" gate="G$1" pin="VBAT"/>
+<pinref part="COIN" gate="G$1" pin="+"/>
+<wire x1="93.98" y1="187.96" x2="111.76" y2="187.96" width="0.1524" layer="91"/>
+</segment>
+</net>
+<net name="RX1" class="0">
+<segment>
+<pinref part="U$1" gate="G$1" pin="0/RX1/T"/>
+<wire x1="48.26" y1="193.04" x2="45.72" y2="193.04" width="0.1524" layer="91"/>
+<label x="45.72" y="193.04" size="1.27" layer="95" rot="R180" xref="yes"/>
+</segment>
+<segment>
+<pinref part="XB1" gate="G$1" pin="DOUT"/>
+<wire x1="-12.7" y1="172.72" x2="-10.16" y2="172.72" width="0.1524" layer="91"/>
+<label x="-10.16" y="172.72" size="1.27" layer="95" xref="yes"/>
+</segment>
+</net>
+<net name="TX1" class="0">
+<segment>
+<pinref part="U$1" gate="G$1" pin="1/TX1/T"/>
+<wire x1="48.26" y1="190.5" x2="45.72" y2="190.5" width="0.1524" layer="91"/>
+<label x="45.72" y="190.5" size="1.27" layer="95" rot="R180" xref="yes"/>
+</segment>
+<segment>
+<pinref part="XB1" gate="G$1" pin="DIN/!CONFIG"/>
+<wire x1="-12.7" y1="175.26" x2="-10.16" y2="175.26" width="0.1524" layer="91"/>
+<label x="-10.16" y="175.26" size="1.27" layer="95" xref="yes"/>
+</segment>
+</net>
+<net name="5V" class="0">
+<segment>
+<pinref part="IC1" gate="G$1" pin="VO"/>
+<wire x1="167.64" y1="182.88" x2="170.18" y2="182.88" width="0.1524" layer="91"/>
+<label x="170.18" y="182.88" size="1.27" layer="95" xref="yes"/>
+</segment>
 <segment>
 <pinref part="U$1" gate="G$1" pin="VIN"/>
@@
 <label x="96.52" y="193.04" size="1.27" layer="95" xref="yes"/>
 </segment>
-<segment>
-<pinref part="X1" gate="-1" pin="S"/>
-<wire x1="142.24" y1="180.34" x2="139.7" y2="180.34" width="0.1524" layer="91"/>
-<label x="139.7" y="180.34" size="1.27" layer="95" rot="R180" xref="yes"/>
-</segment>
-</net>
-<net name="N$9" class="0">
-<segment>
-<junction x="71.12" y="83.82"/>
-</segment>
-</net>
-<net name="N$10" class="0">
-<segment>
-<pinref part="LED1" gate="G$1" pin="A"/>
-<pinref part="R1" gate="G$1" pin="1"/>
-<wire x1="25.4" y1="157.48" x2="27.94" y2="157.48" width="0.1524" layer="91"/>
-</segment>
-</net>
-<net name="N$2" class="0">
-<segment>
-<pinref part="R1" gate="G$1" pin="2"/>
-<pinref part="U$1" gate="G$1" pin="14/A0"/>
-<wire x1="38.1" y1="157.48" x2="48.26" y2="157.48" width="0.1524" layer="91" style="longdash"/>
-</segment>
-</net>
-<net name="N$13" class="0">
-<segment>
-<pinref part="R7" gate="G$1" pin="2"/>
-<pinref part="C1" gate="G$1" pin="3V3"/>
-<wire x1="-30.48" y1="50.8" x2="-30.48" y2="45.72" width="0.1524" layer="91" style="longdash"/>
-</segment>
-</net>
-<net name="N$12" class="0">
-<segment>
-<pinref part="U$1" gate="G$1" pin="VBAT"/>
-<pinref part="COIN" gate="G$1" pin="+"/>
-<wire x1="93.98" y1="187.96" x2="111.76" y2="187.96" width="0.1524" layer="91"/>
-</segment>
-</net>
-<net name="RX1" class="0">
-<segment>
-<pinref part="U$1" gate="G$1" pin="0/RX1/T"/>
-<wire x1="48.26" y1="193.04" x2="45.72" y2="193.04" width="0.1524" layer="91"/>
-<label x="45.72" y="193.04" size="1.27" layer="95" rot="R180" xref="yes"/>
-</segment>
-<segment>
-<pinref part="XB1" gate="G$1" pin="DOUT"/>
-<wire x1="-12.7" y1="172.72" x2="-10.16" y2="172.72" width="0.1524" layer="91"/>
-<label x="-10.16" y="172.72" size="1.27" layer="95" xref="yes"/>
-</segment>
-</net>
-<net name="TX1" class="0">
-<segment>
-<pinref part="U$1" gate="G$1" pin="1/TX1/T"/>
-<wire x1="48.26" y1="190.5" x2="45.72" y2="190.5" width="0.1524" layer="91"/>
-<label x="45.72" y="190.5" size="1.27" layer="95" rot="R180" xref="yes"/>
-</segment>
-<segment>
-<pinref part="XB1" gate="G$1" pin="DIN/!CONFIG"/>
-<wire x1="-12.7" y1="175.26" x2="-10.16" y2="175.26" width="0.1524" layer="91"/>
-<label x="-10.16" y="175.26" size="1.27" layer="95" xref="yes"/>
+</net>
+<net name="N$6" class="0">
+<segment>
+<pinref part="C2" gate="G$1" pin="1"/>
+<wire x1="144.78" y1="180.34" x2="144.78" y2="182.88" width="0.1524" layer="91"/>
+<pinref part="IC1" gate="G$1" pin="VI"/>
+<wire x1="144.78" y1="182.88" x2="147.32" y2="182.88" width="0.1524" layer="91"/>
+<wire x1="144.78" y1="182.88" x2="139.7" y2="182.88" width="0.1524" layer="91"/>
+<junction x="144.78" y="182.88"/>
 </segment>
 </net>
@@
 packages will not be understood (or retained) with this version.
 </note>
+<note version="8.4" severity="warning">
+Since Version 8.4, EAGLE supports properties for SPICE simulation.
+Probes in schematics and SPICE mapping objects found in parts and library devices
+will not be understood with this version. Update EAGLE to the latest version
+for full support of SPICE simulation.
+</note>
 </compatibility>
